File: kicad/test_board/test_board.kicad_pcb (KiCad board)
At the start: 4 copper layers, 40000 x 30000 mm, 9 parts

Commit message: feat: 完善 KiCad 测试载板四层 PCB 设计
- 更新 PCB 为 KiCad 7 格式
- 添加四层板叠层定义 (FR4, ENIG)
- 完善 QFN-48 封装和热过孔
- 添加完整的网络连接和布线
Parts:
- removed ? (x4): , MountingHole:MountingHole_2.2mm_M2
- removed ?: , kicad:QFN-48_7x7mm_P0.5mm
- removed ? (x2): , Capacitor_SMD:C_0402_1005Metric
- removed ?: , Connector_PinHeader_2.54mm:PinHeader_2x05_P2.54mm_Vertical
- removed ?: , Crystal:Crystal_SMD_3215-2Pin_3.2x1.5mm
- added C1: 18pF, Capacitor_SMD:C_0402_1005Metric, F.Cu at (12.0, 10.5)
- added C2: 18pF, Capacitor_SMD:C_0402_1005Metric, F.Cu at (12.0, 5.50)
- added C3: 100nF, Capacitor_SMD:C_0402_1005Metric, F.Cu at (14.0, 11.5)
- added C4: 100nF, Capacitor_SMD:C_0402_1005Metric, F.Cu at (14.0, 18.5)
- added C5: 100nF, Capacitor_SMD:C_0402_1005Metric, F.Cu at (26.0, 11.5)
- added C6: 10uF, Capacitor_SMD:C_0402_1005Metric, F.Cu at (26.0, 18.5)
- added C8: 10uF, Capacitor_SMD:C_0805_2012Metric, F.Cu at (4.50, 6.00)
- added C9: 10uF, Capacitor_SMD:C_0805_2012Metric, F.Cu at (11.5, 6.00)
- added H1: MountingHole, MountingHole:MountingHole_2.2mm_M2, F.Cu at (3.00, 3.00)
- added H2: MountingHole, MountingHole:MountingHole_2.2mm_M2, F.Cu at (37.0, 3.00)
- added H3: MountingHole, MountingHole:MountingHole_2.2mm_M2, F.Cu at (3.00, 27.0)
- added H4: MountingHole, MountingHole:MountingHole_2.2mm_M2, F.Cu at (37.0, 27.0)
- added J1: JTAG, Connector_PinHeader_2.54mm:PinHeader_1x06_P2.54mm_Vertical, F.Cu at (32.0, 4.00)
- added J2: GPIO, Connector_PinHeader_2.54mm:PinHeader_1x08_P2.54mm_Vertical, F.Cu at (8.00, 26.0)
- added R1: 10k, Resistor_SMD:R_0402_1005Metric, F.Cu at (5.00, 22.0)
- added SW1: RESET, Button_Switch_SMD:SW_SPST_TL3342, F.Cu at (8.00, 22.0)
- added U1: PicoRV32, kicad:QFN-48_7x7mm_P0.5mm, F.Cu at (20.0, 15.0)
- added U2: LDO_3V3, Package_TO_SOT_SMD:SOT-23-5, F.Cu at (8.00, 6.00)
- added Y1: 100MHz, Crystal:Crystal_SMD_3215-2Pin_3.2x1.5mm, F.Cu at (12.0, 8.00)
Routing:
- net +3V3: track 0.00 -> 47.4 mm
- net RESETN: track 0.00 -> 20.0 mm
- net CLK: track 0.00 -> 5.81 mm
- net GND: vias 0 -> 8
- added copper zone on In2.Cu, net +3V3
- added copper zone on In1.Cu, net GND
- removed copper zone on In2.Cu, net VDD
- removed copper zone on In1.Cu, net VSS
Other:
- board size 40000 x 30000 mm -> 40 x 30 mm
- rule pad_to_mask_clearance: 0 -> 0.05
- board text added: "40mm x 30mm"
- board text added: "PicoRV32 RISC-V Test Board"
- board text added: "Rev 1.0"
- board text added: "SKY130"
